File: eletronica/ROBOTIC_ARM/ROBOTIC_ARM.kicad_pcb (KiCad board)
At the start: 2 copper layers, 51 x 71.5 mm, 4 parts, among them J1 Conn_01x15_Socket, J2 Conn_01x15_Socket, J3 BORN, J4 RX E TX

Commit message: fix: ajustes na placa
Parts:
- moved J4 38.7 mm to (101.0, 83.0)
- moved J1 27.2 mm to (133.0, 67.4)
- moved J2 21.2 mm to (109.0, 67.4)
- moved J3 2.50 mm to (117.5, 116.5)
Connections:
- J1 pad 1: unconnected-(J1-Pin_1-Pad1) -> /VIN
- J1 pad 13: /VIN -> unconnected-(J1-Pin_13-Pad13)
- J3 pad 1: /VIN -> /GND
- J3 pad 2: /GND -> /VIN
Routing:
- net /VIN: track 27.4 -> 55.5 mm
- net /GND: track 75.7 -> 63.0 mm
- net /RX: track 12.4 -> 8.15 mm
- net /TX: track 12.4 -> 8.15 mm
