File: eletronica/ROBOTIC_ARM/ROBOTIC_ARM.kicad_sch (KiCad schematic)
At the start: 4 parts, among them J1 Conn_01x15_Socket, J2 Conn_01x15_Socket, J3 BORN, J4 RX E TX

Commit message: fix: ajustes na placa
Connections:
- net GND: now also J3.1 (Pin_1); no longer J3.2 (Pin_2)
- net VIN: now also J1.1 (Pin_1), J3.2 (Pin_2); no longer J1.13 (Pin_13), J3.1 (Pin_1)
Changed lines of the file:
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@@
+	(wire
+		(pts
+			(xy 72.39 33.02) (xy 76.2 33.02)
+		)
+		(stroke
+			(width 0)
+			(type default)
+		)
+	)
 	(wire
 		(pts
@@
 		(pts
 			(xy 92.71 76.2) (xy 96.52 76.2)
-		)
-		(stroke
-			(width 0)
-			(type default)
-		)
-	)
-	(wire
-		(pts
-			(xy 71.12 63.5) (xy 76.2 63.5)
 		)
 		(stroke
@@
 		)
 	)
-	(label "GND"
+	(label "VIN"
 		(at 58.42 83.82 0)
 		(effects
@@
 	)
 	(label "VIN"
-		(at 71.12 63.5 0)
+		(at 72.39 33.02 0)
 		(effects
 			(font
@@
 		)
 	)
-	(label "VIN"
+	(label "GND"
 		(at 58.42 81.28 0)
 		(effects
